Commit message: adding d435 plugin

File: piloting_gazebo_simulation/models/mbzirc/geometry.xacro (robot description, xacro)
@@ -37,8 +37,8 @@
     ixy="0.0" ixz="0.0"  iyz="0.0" /> <!-- [kg.m^2] [kg.m^2] [kg.m^2] [kg.m^2] [kg.m^2] [kg.m^2] -->
   </xacro:property>
-  <!--Property cylinder_camera-->
+  <!-- Property cylinder_camera
   <xacro:property name="camera_cylinder">
     <box size="0.1 0.025 0.02"/>
-  </xacro:property>
+  </xacro:property> -->
   <!-- Included URDF Files -->
   <xacro:include filename="$(find robots_description)/urdf/multirotor_base.xacro" />

File: piloting_gazebo_simulation/models/mbzirc/model.xacro (robot description, xacro)
@@ -16,5 +16,10 @@
   <xacro:include filename="$(find robots_description)/urdf/component_snippets.xacro" />
   <!-- Instantiate mbzirc "mechanics" -->
-  <xacro:include filename="$(find robots_description)/models/mbzirc/geometry.xacro" />
+  <xacro:include filename="$(find piloting_gazebo_simulation)/models/mbzirc/geometry.xacro" />
+  <xacro:include filename="$(find realsense_gazebo_plugin)/urdf/d435.urdf.xacro"/>
+  <!-- <link name="base_link" /> -->
+  <sensor_d435 parent="base_link">
+    <origin xyz="0.4 0 0" rpy="0 0 0"/>
+  </sensor_d435>
   <xacro:if value="$(arg enable_gps_plugin)">
     <!-- Instantiate gps plugin. -->
@@ -115,10 +120,4 @@
     </xacro:bag_plugin_macro>
   </xacro:if>
-  <!-- Import macro for realsense-RS200 camera-->
-  <xacro:include filename="$(find realsense_gazebo_plugin)/urdf/realsense-RS200.macro.xacro"/>
-  <!-- Create camera instance -->
-  <xacro:realsense-rs200 prefix="" parent="base_link">
-      <origin xyz="0.22 0 -0.14" rpy="0 0 0" />
-  </xacro:realsense-rs200>
   <!-- <xacro:vi_sensor_depth_macro
     namespace="${namespace}"
